Commit message: feat: deliver Gazebo digital twin baseline

File: ros_ws/src/amr_description/urdf/amr.urdf.xacro (robot description, xacro)
@@ -1,5 +1,5 @@
 <?xml version="1.0"?>
 <robot xmlns:xacro="http://www.ros.org/wiki/xacro" name="portfolio_amr">
-  <xacro:property name="pi" value="3.141592653589793"/>
+  <xacro:property name="wheel_axis_rotation" value="1.5707963267948966"/>
   <xacro:property name="base_length" value="0.55"/>
   <xacro:property name="base_width" value="0.42"/>
@@ -31,14 +31,14 @@
     <link name="${side}_wheel_link">
       <visual>
-        <origin rpy="${pi / 2.0} 0 0"/>
+        <origin rpy="${wheel_axis_rotation} 0 0"/>
         <geometry><cylinder radius="${wheel_radius}" length="${wheel_width}"/></geometry>
         <material name="rubber_black"/>
       </visual>
       <collision>
-        <origin rpy="${pi / 2.0} 0 0"/>
+        <origin rpy="${wheel_axis_rotation} 0 0"/>
         <geometry><cylinder radius="${wheel_radius}" length="${wheel_width}"/></geometry>
       </collision>
       <inertial>
-        <origin rpy="${pi / 2.0} 0 0"/>
+        <origin rpy="${wheel_axis_rotation} 0 0"/>
         <mass value="${wheel_mass}"/>
         <inertia
@@ -127,5 +127,5 @@
       <update_rate>15</update_rate>
       <lidar>
-        <scan><horizontal><samples>720</samples><resolution>1</resolution><min_angle>-${pi}</min_angle><max_angle>${pi}</max_angle></horizontal></scan>
+        <scan><horizontal><samples>720</samples><resolution>1</resolution><min_angle>-${3.141592653589793}</min_angle><max_angle>${3.141592653589793}</max_angle></horizontal></scan>
         <range><min>0.12</min><max>12.0</max><resolution>0.01</resolution></range>
         <noise><type>gaussian</type><mean>0.0</mean><stddev>0.005</stddev></noise>
